File: dsplolo.brd (EAGLE design)
At the start: 100 x 80 mm, 42 parts, among them IC1 AD8608R, T1 BC847, U1 TDA7293V, U2 TDA7293V, U3 TDA7293V

Commit message: latest
Parts:
- removed U1, U2, U3: TDA7293V, TDA7293V:TDA7293V
- added C21, C22, C25, C27, C28, C29, C33, C42, C43, C48: 100n, resistor:C1206
- added C23, C24, C26, C30, C31, C32, C44, C45: 10u, resistor:C1206
- added C34: 56n, resistor:C1206
- added C35: 3n3, resistor:C1206
- added C36, C37: 22p, resistor:C1206
- added C38, C40, C49, C50: 4u7, resistor:C1206
- added C39, C41: 100p, resistor:C1206
- added IC2: REG1117, burr-brown:SOT223
- added IC3: 24AA256SM, microchip:SO-08M
- added JP1, JP2: (no value), pinhead:1X10
- added Q1: 12.288M, crystal:HC49UP
- added R17: 1k, rcl:R1206
- added R18: 18k, rcl:R1206
- added R19, R32, R33: 6k8, rcl:R1206
- added R20: 475, rcl:R1206
- added R21: 100, rcl:R1206
- added R22, R27: 49k9, rcl:R1206
- added R23, R24, R25, R26, R28, R29, R30, R31: ?, rcl:R1206
- added S1, S2: 219-04, switch-dil:CTS-219-04
- added X1: INPUT, adafruit:STX3100
- added X2: OUTPUT1, adafruit:STX3100
- added X3: OUTPUT2, adafruit:STX3100
- added X4: MINI-USB-UX60A-MB-5ST, con-hirose:UX60A-MB-5ST
- T1: value BC847 -> (none); device transistor:SOT23 -> transistor:SOT23-BEC
- moved R13 229.6 mm to (55.9, 55.9), turned to 180 degrees
- moved R14 226.8 mm to (49.5, 55.2), turned to 270 degrees
- moved T1 225.2 mm to (66.7, 26.7), turned to 90 degrees
- moved R15 221.2 mm to (21.6, 39.4), turned to 180 degrees
- moved C17 221.0 mm to (46.4, 55.2), turned to 270 degrees
- moved C20 220.2 mm to (17.8, 38.1), turned to 270 degrees
- moved C16 218.0 mm to (50.2, 50.2), turned to 270 degrees
- moved R11 215.1 mm to (21.6, 33.0), turned to 180 degrees
- moved C18 214.8 mm to (26.7, 39.4), turned to 180 degrees
- moved C19 212.1 mm to (26.7, 36.8), turned to 180 degrees
- moved C14 209.1 mm to (26.7, 33.0), turned to 180 degrees
- moved C13 207.2 mm to (26.7, 30.5), turned to 180 degrees
- moved R16 207.1 mm to (15.2, 38.1), turned to 90 degrees
- moved C15 207.1 mm to (17.8, 31.8), turned to 270 degrees
- moved R10 206.9 mm to (48.9, 42.5), turned to 90 degrees
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Connections:
- removed net V+: IC1.4
- removed net V-: IC1.11
- new net +3V3: C21.2, C23.2, C25.2, C26.2, C27.1, C35.1, C43.1, C45.1, C48.1, IC1.4, IC2.2, IC3.8, R17.2, R19.2, R20.2, R32.2, R33.2, T1.E, U$1.18, U$1.34, U$1.36, U$1.39, U$1.48, U$1.6
- new net +5V: C42.1, C44.1, IC2.3, JP2.1, X4.1
- new net MP0: JP2.2, U$1.11
- new net MP1: JP2.3, U$1.10
- new net MP10: JP1.7, U$1.16
- new net MP11: JP1.6, U$1.19
- new net MP2: JP2.4, U$1.29
- new net MP3: JP2.5, U$1.28
- new net MP4: JP2.6, U$1.8
- new net MP5: JP2.7, U$1.9
- new net MP6: JP2.8, U$1.15
- new net MP7: JP2.9, U$1.14
- new net MP8: JP1.9, U$1.27
- new net MP9: JP1.8, U$1.26
- new net N$21: R18.2, U$1.3
- new net N$22: C22.1, C24.1, T1.C, U$1.13, U$1.24
- new net N$23: R17.1, T1.B, U$1.17
- new net N$24: R1.1, U$1.46
- new net N$25: R5.1, U$1.45
- new net N$26: R9.1, U$1.44
- new net N$27: R13.1, U$1.43
- new net N$28: C32.2, C33.2, U$1.47
- new net N$29: C37.2, Q1.1, U$1.32
- new net N$30: C29.2, C31.2, U$1.41
- new net N$31: C28.2, C30.2, U$1.40
- new net N$32: C34.2, C35.2, U$1.35
- new net N$33: C34.1, R20.1
- new net N$34: C36.2, Q1.2, R21.1
- new net N$35: R21.2, U$1.31
- new net N$36: R23.1, S1.4
- new net N$37: C38.1, C39.1, C50.1, R22.2, X1.5
- new net N$38: C38.2, C50.2, S1.5, S1.6, S1.7, S1.8
- new net N$39: R24.1, S1.3
- new net N$40: R25.1, S1.2
- new net N$41: R26.1, S1.1
- new net N$42: R23.2, R24.2, R25.2, R26.2, U$1.2
- new net N$44: C40.1, C41.1, C49.1, R27.2, X1.3
- new net N$45: C40.2, C49.2, S2.5, S2.6, S2.7, S2.8
- new net N$46: R28.1, S2.4
- new net N$47: R29.1, S2.3
- new net N$48: R30.1, S2.2
- new net N$49: R31.1, S2.1
- new net N$50: R28.2, R29.2, R30.2, R31.2, U$1.4
- new net NRST: JP1.1, R19.1, U$1.5
- new net SCL: IC3.6, JP1.4, R32.1, U$1.23
- new net SDA: IC3.5, JP1.5, R33.1, U$1.22
- new net WB: JP1.2, U$1.20
- new net WP: IC3.7, JP1.3, U$1.21
- net GND: now also C21.1, C22.2, C23.1, C24.2, C25.1, C26.1, C27.2, C28.1, C29.1, C30.1, C31.1, C32.1, C33.1, C36.1, C37.1, C39.2, C41.2, C42.2, C43.2, C44.2, C45.2, C48.2, IC1.11, IC2.1, IC3.1, IC3.2, IC3.3, IC3.4, JP1.10, JP2.10, R18.1, R22.1, R27.1, U$1.1, U$1.12, U$1.25, U$1.30, U$1.33, U$1.37, U$1.38, U$1.42, U$1.7, X1.1, X2.1, X3.1, X4.5
- net N$12: now also X3.5
- net N$17: now also X3.3
- net N$3: now also X2.5
- net N$7: now also X2.3
Routing:
- net +3V3: track 0.00 -> 238.6 mm, vias 0 -> 6
- net GND: track 0.00 -> 158.7 mm, vias 0 -> 68
- net +5V: track 0.00 -> 111.3 mm, vias 0 -> 2
- net N$24: track 0.00 -> 50.4 mm, vias 0 -> 2
- net NRST: track 0.00 -> 49.4 mm, vias 0 -> 1
- net WP: track 0.00 -> 47.4 mm
- net N$42: track 0.00 -> 47.2 mm, vias 0 -> 2
- net N$25: track 0.00 -> 43.5 mm, vias 0 -> 2
- net MP10: track 0.00 -> 40.8 mm, vias 0 -> 1
- net MP7: track 0.00 -> 38.7 mm, vias 0 -> 1
- net MP5: track 0.00 -> 38.5 mm, vias 0 -> 1
- net MP6: track 0.00 -> 37.7 mm, vias 0 -> 1
- net MP8: track 0.00 -> 37.1 mm, vias 0 -> 1
- net SCL: track 0.00 -> 37.0 mm, vias 0 -> 2
- net MP9: track 0.00 -> 36.3 mm
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- added copper zone on layer 1, net GND
- added copper zone on layer 15, net GND
- added copper zone on layer 16, net GND
- added copper zone on layer 2, net GND
Other:
- board size 100 x 80 mm -> 94.9 x 62.2 mm
