File: dsplolo.sch (EAGLE design)
At the start: 42 parts, among them IC1 AD8608R, T1 BC847, U1 TDA7293V, U2 TDA7293V, U3 TDA7293V

Commit message: latest
Parts:
- removed U1, U2, U3: TDA7293V, TDA7293V:TDA7293V
- added C21, C22, C25, C27, C28, C29, C33, C42, C43, C48: 100n, resistor:C-EUC1206
- added C23, C24, C26, C30, C31, C32, C44, C45: 10u, resistor:C-EUC1206
- added C34: 56n, resistor:C-EUC1206
- added C35: 3n3, resistor:C-EUC1206
- added C36, C37: 22p, resistor:C-EUC1206
- added C38, C40, C49, C50: 4u7, resistor:C-EUC1206
- added C39, C41: 100p, resistor:C-EUC1206
- added IC2: REG1117, burr-brown:REG1117
- added IC3: 24AA256SM, microchip:24AA128SM
- added JP1, JP2: (no value), pinhead:PINHD-1X10
- added Q1: 12.288M, crystal:CRYSTALHC49UP
- added R17: 1k, rcl:R-EU_R1206
- added R18: 18k, rcl:R-EU_R1206
- added R19, R32, R33: 6k8, rcl:R-EU_R1206
- added R20: 475, rcl:R-EU_R1206
- added R21: 100, rcl:R-EU_R1206
- added R22, R27: 49k9, rcl:R-EU_R1206
- added R23, R24, R25, R26, R28, R29, R30, R31: ?, rcl:R-EU_R1206
- added S1, S2: 219-04, switch-dil:219-04
- added X1: INPUT, adafruit:STEREOJACK
- added X2: OUTPUT1, adafruit:STEREOJACK
- added X3: OUTPUT2, adafruit:STEREOJACK
- added X4: MINI-USB-UX60A-MB-5ST, con-hirose:MINI-USB-UX60A-MB-5ST
- T1: value BC847 -> (none); device transistor:BC847 -> transistor:BC857C-PNP-SOT23-BEC
Connections:
- new net +3V3: C21.2, C23.2, C25.2, C26.2, C27.1, C35.1, C43.1, C45.1, C48.1, IC1G$1.V+, IC2.VOUT, IC3.VCC, R17.2, R19.2, R20.2, R32.2, R33.2, T1.E, U$1.AVDD, U$1.AVDD@1, U$1.IOVDD, U$1.PLL_MODE1, U$1.PVDD, U$1.SELFBOOT
- new net +5V: C42.1, C44.1, IC2.VIN, JP2.1, X4.1
- new net MP0: JP2.2, U$1.MP0
- new net MP1: JP2.3, U$1.MP1
- new net MP10: JP1.7, U$1.MP10
- new net MP11: JP1.6, U$1.MP11
- new net MP2: JP2.4, U$1.MP2
- new net MP3: JP2.5, U$1.MP3
- new net MP4: JP2.6, U$1.MP4
- new net MP5: JP2.7, U$1.MP5
- new net MP6: JP2.8, U$1.MP6
- new net MP7: JP2.9, U$1.MP7
- new net MP8: JP1.9, U$1.MP8
- new net MP9: JP1.8, U$1.MP9
- new net N$21: R18.2, U$1.ADC_RES
- new net N$22: C22.1, C24.1, T1.C, U$1.DVDD, U$1.DVDD@1
- new net N$23: R17.1, T1.B, U$1.VDRIVE
- new net N$24: R1.1, U$1.VOUT0
- new net N$25: R5.1, U$1.VOUT1
- new net N$26: R9.1, U$1.VOUT2
- new net N$27: R13.1, U$1.VOUT3
- new net N$28: C32.2, C33.2, U$1.FILTA
- new net N$29: C37.2, Q1.1, U$1.MCLOCKI
- new net N$30: C29.2, C31.2, U$1.FILTD
- new net N$31: C28.2, C30.2, U$1.CM
- new net N$32: C34.2, C35.2, U$1.PLL_LF
- new net N$33: C34.1, R20.1
- new net N$34: C36.2, Q1.2, R21.1
- new net N$35: R21.2, U$1.OSCO
- new net N$36: R23.1, S1.4
- new net N$37: C38.1, C39.1, C50.1, R22.2, X1.5
- new net N$38: C38.2, C50.2, S1.5, S1.6, S1.7, S1.8
- new net N$39: R24.1, S1.3
- new net N$40: R25.1, S1.2
- new net N$41: R26.1, S1.1
- new net N$42: R23.2, R24.2, R25.2, R26.2, U$1.ADC0
- new net N$44: C40.1, C41.1, C49.1, R27.2, X1.3
- new net N$45: C40.2, C49.2, S2.5, S2.6, S2.7, S2.8
- new net N$46: R28.1, S2.4
- new net N$47: R29.1, S2.3
- new net N$48: R30.1, S2.2
- new net N$49: R31.1, S2.1
- new net N$50: R28.2, R29.2, R30.2, R31.2, U$1.ADC1
- new net NRST: JP1.1, R19.1, U$1./RESET
- new net SCL: IC3.SCL, JP1.4, R32.1, U$1.SCL/CCLK
- new net SDA: IC3.SDA, JP1.5, R33.1, U$1.SDA/COUT
- new net WB: JP1.2, U$1.ADR1/CDATA/WB
- new net WP: IC3.WP, JP1.3, U$1.CLATCH/WP
- net GND: now also C21.1, C22.2, C23.1, C24.2, C25.1, C26.1, C27.2, C28.1, C29.1, C30.1, C31.1, C32.1, C33.1, C36.1, C37.1, C39.2, C41.2, C42.2, C43.2, C44.2, C45.2, C48.2, IC1G$1.V-, IC2.GND, IC3.A0, IC3.A1, IC3.A2, IC3.GND, JP1.10, JP2.10, R18.1, R22.1, R27.1, U$1.ADR0, U$1.AGND, U$1.AGND@1, U$1.AGND@2, U$1.DGND, U$1.DGND@1, U$1.PGND, U$1.PLL_MODE0, U$1.RSVD, X1.1, X2.1, X3.1, X4.5
- net N$12: now also X3.5
- net N$17: now also X3.3
- net N$3: now also X2.5
- net N$7: now also X2.3
